Commit message: 1.给所有link添加了<gazebo>下的摩擦,Kp等 2.添加了执行器 3.添加了差速运动插件 4.imu还没有完成

File: models/mcar_urdf/model.urdf (robot description, URDF)
Before this commit: robot mcar_urdf, 1 links, 0 joints
Links:
- added link laser, mass 1e-3; collision cylinder length=0.1 radius=0.08; visual cylinder length=0.1 radius=0.08
- added link left_wheel, mass 0.01; collision cylinder length=0.1 radius=0.15; visual cylinder length=0.1 radius=0.15
- added link right_wheel, mass 0.01; collision cylinder length=0.1 radius=0.15; visual cylinder length=0.1 radius=0.15
- link chassis: mass 1.0 -> 0.2; geometry collision box size=0.5 0.3 0.2; collision sphere radius=0.05
Joints:
- added joint laser2bass: type fixed, parent chassis, child laser, origin xyz=0.15 0.0 0.35 rpy=0.0 0.0 0.0, axis 0.0 0.0 0.0
- added joint left_joint: type continuous, parent chassis, child left_wheel, origin xyz=0.15 0.21 0.15 rpy=0.0 0.0 0.0, axis 0.0 1.0 0.0
- added joint right_joint: type continuous, parent chassis, child right_wheel, origin xyz=0.15 -0.21 0.15 rpy=0.0 0.0 0.0, axis 0.0 1.0 0.0

Commit message: 1.添加了imu 2.ros_control还没有完全理解

File: models/mcar_urdf/model.urdf (robot description, URDF)
Before this commit: robot mcar_urdf, 4 links, 3 joints
Links:
- added link imu_link, mass 1e-6; collision box size=0.1 0.1 0.02; visual box size=0.1 0.1 0.02
Joints:
- removed joint laser2bass
- added joint imu_joint: type fixed, parent chassis, child imu_link, origin xyz=0.0 0.0 0.31 rpy=0.0 0.0 0.0, axis 0.0 0.0 0.0, limit lower=0.0 upper=0.0 effort=0.0 velocity=0.0
- added joint laser_joint: type fixed, parent chassis, child laser, origin xyz=0.15 0.0 0.35 rpy=0.0 0.0 0.0, axis 0.0 0.0 0.0
